File: qlexternal512kram_MIX.kicad_sch (KiCad schematic)
At the start: 14 parts, among them J1 QL_SLOT_DIN41612_CARD, J2 QL_SLOT_DIN41612_CARD, SW1 SW_DIP_x02, SW2 SW_SPDT, U1 HM628512BLFP-7, U2 GAL16V8B-25QP, U3 LM1117-5.0

Commit message: WiP: ultimos cambios locales antes de merge
Parts:
- U1: footprint Package_SO:SSOP-32_11.305x20.495mm_P1.27mm -> Package_SO:SOP-32_11.305x20.495mm_P1.27mm
